Commit message: got stls to launch in rviz, next I want to make a custom launch file for rviz

File: src/Goddard/goddard_description/urdf/goddard.urdf (robot description, URDF)
Before this commit: robot goddard, 2 links, 1 joints
Links:
- link body: geometry visual mesh filename=package://goddard_description/meshes/body.stl scale=0.01 0.01 0.01
Joints:
- removed joint base_to_right_leg
- added joint body_to_base_link: type fixed, parent base_link, child body
