Commit message: working on getting gazebo to spawn goddard

File: src/Goddard/goddard_description/urdf/goddard.urdf.xacro (robot description, xacro)
@@ -8,4 +8,13 @@
                     scale="0.001 0.001 0.001" />
             </geometry>
+            <collision>
+                <mesh filename="package://goddard_description/meshes/body.stl"
+                    scale="0.001 0.001 0.001" />
+            </collision>
+            <inertial>
+                <mass value="6.738" />
+                <inertia ixx="16.22" ixy="0.000105591" ixz="0.000054509" iyy="44.31"
+                    iyz="-0.014467893" izz="50.43" />
+            </inertial>
         </visual>
     </link>
@@ -15,4 +24,5 @@
         <origin xyz="0 0 0.1226" />
     </joint>
+    <!-- Front Left Components  -->
     <link name="front_left_hip">
         <visual>
@@ -21,4 +31,12 @@
                     scale="0.001 0.001 0.001" />
             </geometry>
+            <collision>
+                <mesh filename="package://goddard_description/meshes/hip.stl"
+                    scale="0.001 0.001 0.001" />
+            </collision>
+            <inertial>
+                <mass value="0.2" />
+                <inertia ixx="0.4" ixy="0.0" ixz="0.0" iyy="0.4" iyz="0.0" izz="0.2" />
+            </inertial>
         </visual>
     </link>
@@ -36,4 +54,12 @@
                     scale="0.001 0.001 0.001" />
             </geometry>
+            <collision>
+                <mesh filename="package://goddard_description/meshes/femur.stl"
+                    scale="0.001 0.001 0.001" />
+            </collision>
+            <inertial>
+                <mass value="0.2" />
+                <inertia ixx="0.4" ixy="0.0" ixz="0.0" iyy="0.4" iyz="0.0" izz="0.2" />
+            </inertial>
             <origin xyz="-0.0246 0 -0.02835" />
         </visual>
@@ -52,4 +78,12 @@
                     scale="0.001 0.001 0.001" />
             </geometry>
+            <collision>
+                <mesh filename="package://goddard_description/meshes/tibia.stl"
+                    scale="0.001 0.001 0.001" />
+            </collision>
+            <inertial>
+                <mass value="0.2" />
+                <inertia ixx="0.4" ixy="0.0" ixz="0.0" iyy="0.4" iyz="0.0" izz="0.2" />
+            </inertial>
             <origin xyz="0.01861 0 -0.02100" />
         </visual>
@@ -62,4 +96,5 @@
         <limit lower="-1.571" upper="1.571" effort="1000" velocity="0.5" />
     </joint>
+    <!-- Front Right Components -->
     <link name="front_right_hip">
         <visual>
@@ -68,4 +103,12 @@
                     scale="0.001 0.001 0.001" />
             </geometry>
+            <collision>
+                <mesh filename="package://goddard_description/meshes/hip.stl"
+                    scale="0.001 0.001 0.001" />
+            </collision>
+            <inertial>
+                <mass value="0.2" />
+                <inertia ixx="0.4" ixy="0.0" ixz="0.0" iyy="0.4" iyz="0.0" izz="0.2" />
+            </inertial>
             <origin xyz="0 0 0" rpy="0 0 3.142" />
         </visual>
@@ -84,4 +127,12 @@
                     scale="0.001 0.001 0.001" />
             </geometry>
+            <collision>
+                <mesh filename="package://goddard_description/meshes/femur.stl"
+                    scale="0.001 0.001 0.001" />
+            </collision>
+            <inertial>
+                <mass value="0.2" />
+                <inertia ixx="0.4" ixy="0.0" ixz="0.0" iyy="0.4" iyz="0.0" izz="0.2" />
+            </inertial>
             <origin xyz="-0.0246 0 -0.02835" />
         </visual>
@@ -100,4 +151,12 @@
                     scale="0.001 0.001 0.001" />
             </geometry>
+            <collision>
+                <mesh filename="package://goddard_description/meshes/tibia.stl"
+                    scale="0.001 0.001 0.001" />
+            </collision>
+            <inertial>
+                <mass value="0.2" />
+                <inertia ixx="0.4" ixy="0.0" ixz="0.0" iyy="0.4" iyz="0.0" izz="0.2" />
+            </inertial>
             <origin xyz="0.01861 0 -0.02100" />
         </visual>
@@ -110,4 +169,5 @@
         <limit lower="-1.571" upper="1.571" effort="1000" velocity="0.5" />
     </joint>
+    <!-- Back Left Components -->
     <link name="back_left_hip">
         <visual>
@@ -116,4 +176,12 @@
                     scale="0.001 0.001 0.001" />
             </geometry>
+            <collision>
+                <mesh filename="package://goddard_description/meshes/hip.stl"
+                    scale="0.001 0.001 0.001" />
+            </collision>
+            <inertial>
+                <mass value="0.2" />
+                <inertia ixx="0.4" ixy="0.0" ixz="0.0" iyy="0.4" iyz="0.0" izz="0.2" />
+            </inertial>
             <origin xyz="0 0 0" rpy="0 0 3.142" />
         </visual>
@@ -132,4 +200,12 @@
                     scale="0.001 0.001 0.001" />
             </geometry>
+            <collision>
+                <mesh filename="package://goddard_description/meshes/femur.stl"
+                    scale="0.001 0.001 0.001" />
+            </collision>
+            <inertial>
+                <mass value="0.2" />
+                <inertia ixx="0.4" ixy="0.0" ixz="0.0" iyy="0.4" iyz="0.0" izz="0.2" />
+            </inertial>
             <origin xyz="-0.0246 0 -0.02835" />
         </visual>
@@ -148,4 +224,12 @@
                     scale="0.001 0.001 0.001" />
             </geometry>
+            <collision>
+                <mesh filename="package://goddard_description/meshes/tibia.stl"
+                    scale="0.001 0.001 0.001" />
+            </collision>
+            <inertial>
+                <mass value="0.2" />
+                <inertia ixx="0.4" ixy="0.0" ixz="0.0" iyy="0.4" iyz="0.0" izz="0.2" />
+            </inertial>
             <origin xyz="0.01861 0 -0.02100" />
         </visual>
@@ -158,4 +242,5 @@
         <limit lower="-1.571" upper="1.571" effort="1000" velocity="0.5" />
     </joint>
+    <!-- Back Right Components -->
     <link name="back_right_hip">
         <visual>
@@ -164,4 +249,12 @@
                     scale="0.001 0.001 0.001" />
             </geometry>
+            <collision>
+                <mesh filename="package://goddard_description/meshes/hip.stl"
+                    scale="0.001 0.001 0.001" />
+            </collision>
+            <inertial>
+                <mass value="0.2" />
+                <inertia ixx="0.4" ixy="0.0" ixz="0.0" iyy="0.4" iyz="0.0" izz="0.2" />
+            </inertial>
             <origin xyz="0 0 0" rpy="0 0 3.142" />
         </visual>
@@ -180,4 +273,12 @@
                     scale="0.001 0.001 0.001" />
             </geometry>
+            <collision>
+                <mesh filename="package://goddard_description/meshes/femur.stl"
+                    scale="0.001 0.001 0.001" />
+            </collision>
+            <inertial>
+                <mass value="0.2" />
+                <inertia ixx="0.4" ixy="0.0" ixz="0.0" iyy="0.4" iyz="0.0" izz="0.2" />
+            </inertial>
             <origin xyz="-0.0246 0 -0.02835" />
         </visual>
@@ -196,4 +297,12 @@
                     scale="0.001 0.001 0.001" />
             </geometry>
+            <collision>
+                <mesh filename="package://goddard_description/meshes/tibia.stl"
+                    scale="0.001 0.001 0.001" />
+            </collision>
+            <inertial>
+                <mass value="0.2" />
+                <inertia ixx="0.4" ixy="0.0" ixz="0.0" iyy="0.4" iyz="0.0" izz="0.2" />
+            </inertial>
             <origin xyz="0.01861 0 -0.02100" />
         </visual>
