Commit message: got robot to show up in sim, gonna add the plugins soon

File: src/Goddard/goddard_description/urdf/goddard.urdf.xacro (robot description, xacro)
@@ -1,20 +1,22 @@
 <?xml version="1.0"?>
-<robot name="goddard">
+<robot xmlns:xacro="http://www.ros.org/wiki/xacro" name="goddard">
     <link name="base_link" />
     <link name="body">
-        <visual>
-            <geometry>
-                <mesh filename="package://goddard_description/meshes/body.stl"
-                    scale="0.001 0.001 0.001" />
-            </geometry>
-            <collision>
-                <mesh filename="package://goddard_description/meshes/body.stl"
-                    scale="0.001 0.001 0.001" />
-            </collision>
-            <inertial>
-                <mass value="6.738" />
-                <inertia ixx="16.22" ixy="0.000105591" ixz="0.000054509" iyy="44.31"
-                    iyz="-0.014467893" izz="50.43" />
-            </inertial>
+        <inertial>
+            <mass value="1" />
+            <inertia ixx="0.1" ixy="0" ixz="0" iyy="0.1"
+                iyz="0" izz="0.1" />
+        </inertial>
+        <collision>
+            <geometry>
+                <mesh filename="file://$(find goddard_description)/meshes/body.stl"
+                    scale="0.001 0.001 0.001" />
+            </geometry>
+        </collision>
+        <visual>
+            <geometry>
+                <mesh filename="file://$(find goddard_description)/meshes/body.stl"
+                    scale="0.001 0.001 0.001" />
+            </geometry>
         </visual>
     </link>
@@ -22,21 +24,24 @@
         <parent link="base_link" />
         <child link="body" />
-        <origin xyz="0 0 0.1226" />
+        <origin xyz="0 0 0.1226" rpy="0 0 0" />
     </joint>
     <!-- Front Left Components  -->
     <link name="front_left_hip">
-        <visual>
-            <geometry>
-                <mesh filename="package://goddard_description/meshes/hip.stl"
-                    scale="0.001 0.001 0.001" />
-            </geometry>
-            <collision>
-                <mesh filename="package://goddard_description/meshes/hip.stl"
-                    scale="0.001 0.001 0.001" />
-            </collision>
-            <inertial>
-                <mass value="0.2" />
-                <inertia ixx="0.4" ixy="0.0" ixz="0.0" iyy="0.4" iyz="0.0" izz="0.2" />
-            </inertial>
+        <inertial>
+            <mass value="1" />
+            <inertia ixx="0.1" ixy="0" ixz="0" iyy="0.1"
+                iyz="0" izz="0.1" />
+        </inertial>
+        <collision>
+            <geometry>
+                <mesh filename="file://$(find goddard_description)/meshes/hip.stl"
+                    scale="0.001 0.001 0.001" />
+            </geometry>
+        </collision>
+        <visual>
+            <geometry>
+                <mesh filename="file://$(find goddard_description)/meshes/hip.stl"
+                    scale="0.001 0.001 0.001" />
+            </geometry>
         </visual>
     </link>
@@ -44,23 +49,27 @@
         <parent link="body" />
         <child link="front_left_hip" />
-        <origin xyz="0.07900 0.05713 0.003000" />
+        <origin xyz="0.07900 0.05713 0.003000" rpy="0 0 0" />
         <axis xyz="1 0 0" />
         <limit lower="-1.571" upper="1.571" effort="1000" velocity="0.5" />
     </joint>
     <link name="front_left_femur">
-        <visual>
-            <geometry>
-                <mesh filename="package://goddard_description/meshes/femur.stl"
-                    scale="0.001 0.001 0.001" />
-            </geometry>
-            <collision>
-                <mesh filename="package://goddard_description/meshes/femur.stl"
-                    scale="0.001 0.001 0.001" />
-            </collision>
-            <inertial>
-                <mass value="0.2" />
-                <inertia ixx="0.4" ixy="0.0" ixz="0.0" iyy="0.4" iyz="0.0" izz="0.2" />
-            </inertial>
-            <origin xyz="-0.0246 0 -0.02835" />
+        <inertial>
+            <mass value="1" />
+            <inertia ixx="0.1" ixy="0" ixz="0" iyy="0.1"
+                iyz="0" izz="0.1" />
+        </inertial>
+        <collision>
+            <geometry>
+                <mesh filename="file://$(find goddard_description)/meshes/femur.stl"
+                    scale="0.001 0.001 0.001" />
+            </geometry>
+            <origin xyz="-0.0246 0 -0.02835" rpy="0 0 0" />
+        </collision>
+        <visual>
+            <geometry>
+                <mesh filename="file://$(find goddard_description)/meshes/femur.stl"
+                    scale="0.001 0.001 0.001" />
+            </geometry>
+            <origin xyz="-0.0246 0 -0.02835" rpy="0 0 0" />
         </visual>
     </link>
@@ -68,23 +77,27 @@
         <parent link="front_left_hip" />
         <child link="front_left_femur" />
-        <origin xyz="0 0.03558 -0.00469" />
+        <origin xyz="0 0.03558 -0.00469" rpy="0 0 0" />
         <axis xyz="0 -1 0" />
         <limit lower="-1.571" upper="1.571" effort="1000" velocity="0.5" />
     </joint>
     <link name="front_left_tibia">
-        <visual>
-            <geometry>
-                <mesh filename="package://goddard_description/meshes/tibia.stl"
-                    scale="0.001 0.001 0.001" />
-            </geometry>
-            <collision>
-                <mesh filename="package://goddard_description/meshes/tibia.stl"
-                    scale="0.001 0.001 0.001" />
-            </collision>
-            <inertial>
-                <mass value="0.2" />
-                <inertia ixx="0.4" ixy="0.0" ixz="0.0" iyy="0.4" iyz="0.0" izz="0.2" />
-            </inertial>
-            <origin xyz="0.01861 0 -0.02100" />
+        <inertial>
+            <mass value="1" />
+            <inertia ixx="0.1" ixy="0" ixz="0" iyy="0.1"
+                iyz="0" izz="0.1" />
+        </inertial>
+        <collision>
+            <geometry>
+                <mesh filename="file://$(find goddard_description)/meshes/tibia.stl"
+                    scale="0.001 0.001 0.001" />
+            </geometry>
+            <origin xyz="0.01861 0 -0.02100" rpy="0 0 0" />
+        </collision>
+        <visual>
+            <geometry>
+                <mesh filename="file://$(find goddard_description)/meshes/tibia.stl"
+                    scale="0.001 0.001 0.001" />
+            </geometry>
+            <origin xyz="0.01861 0 -0.02100" rpy="0 0 0" />
         </visual>
     </link>
@@ -92,5 +105,5 @@
         <parent link="front_left_femur" />
         <child link="front_left_tibia" />
-        <origin xyz="-0.05367 0 -0.05261" />
+        <origin xyz="-0.05367 0 -0.05261" rpy="0 0 0" />
         <axis xyz="0 -1 0" />
         <limit lower="-1.571" upper="1.571" effort="1000" velocity="0.5" />
@@ -98,17 +111,21 @@
     <!-- Front Right Components -->
     <link name="front_right_hip">
-        <visual>
-            <geometry>
-                <mesh filename="package://goddard_description/meshes/hip.stl"
-                    scale="0.001 0.001 0.001" />
-            </geometry>
-            <collision>
-                <mesh filename="package://goddard_description/meshes/hip.stl"
-                    scale="0.001 0.001 0.001" />
-            </collision>
-            <inertial>
-                <mass value="0.2" />
-                <inertia ixx="0.4" ixy="0.0" ixz="0.0" iyy="0.4" iyz="0.0" izz="0.2" />
-            </inertial>
+        <inertial>
+            <mass value="1" />
+            <inertia ixx="0.1" ixy="0" ixz="0" iyy="0.1"
+                iyz="0" izz="0.1" />
+        </inertial>
+        <collision>
+            <geometry>
+                <mesh filename="file://$(find goddard_description)/meshes/hip.stl"
+                    scale="0.001 0.001 0.001" />
+            </geometry>
+            <origin xyz="0 0 0" rpy="0 0 3.142" />
+        </collision>
+        <visual>
+            <geometry>
+                <mesh filename="file://$(find goddard_description)/meshes/hip.stl"
+                    scale="0.001 0.001 0.001" />
+            </geometry>
             <origin xyz="0 0 0" rpy="0 0 3.142" />
         </visual>
@@ -117,23 +134,27 @@
         <parent link="body" />
         <child link="front_right_hip" />
-        <origin xyz="0.07900 -0.05713 0.003000" />
+        <origin xyz="0.07900 -0.05713 0.003000" rpy="0 0 0" />
         <axis xyz="-1 0 0" />
         <limit lower="-1.571" upper="1.571" effort="1000" velocity="0.5" />
     </joint>
     <link name="front_right_femur">
-        <visual>
-            <geometry>
-                <mesh filename="package://goddard_description/meshes/femur.stl"
-                    scale="0.001 0.001 0.001" />
-            </geometry>
-            <collision>
-                <mesh filename="package://goddard_description/meshes/femur.stl"
-                    scale="0.001 0.001 0.001" />
-            </collision>
-            <inertial>
-                <mass value="0.2" />
-                <inertia ixx="0.4" ixy="0.0" ixz="0.0" iyy="0.4" iyz="0.0" izz="0.2" />
-            </inertial>
-            <origin xyz="-0.0246 0 -0.02835" />
+        <inertial>
+            <mass value="1" />
+            <inertia ixx="0.1" ixy="0" ixz="0" iyy="0.1"
+                iyz="0" izz="0.1" />
+        </inertial>
+        <collision>
+            <geometry>
+                <mesh filename="file://$(find goddard_description)/meshes/femur.stl"
+                    scale="0.001 0.001 0.001" />
+            </geometry>
+            <origin xyz="-0.0246 0 -0.02835" rpy="0 0 0" />
+        </collision>
+        <visual>
+            <geometry>
+                <mesh filename="file://$(find goddard_description)/meshes/femur.stl"
+                    scale="0.001 0.001 0.001" />
+            </geometry>
+            <origin xyz="-0.0246 0 -0.02835" rpy="0 0 0" />
         </visual>
     </link>
@@ -141,23 +162,27 @@
         <parent link="front_right_hip" />
         <child link="front_right_femur" />
-        <origin xyz="0 -0.03558 -0.00469" />
+        <origin xyz="0 -0.03558 -0.00469" rpy="0 0 0" />
         <axis xyz="0 -1 0" />
         <limit lower="-1.571" upper="1.571" effort="1000" velocity="0.5" />
     </joint>
     <link name="front_right_tibia">
-        <visual>
-            <geometry>
-                <mesh filename="package://goddard_description/meshes/tibia.stl"
-                    scale="0.001 0.001 0.001" />
-            </geometry>
-            <collision>
-                <mesh filename="package://goddard_description/meshes/tibia.stl"
-                    scale="0.001 0.001 0.001" />
-            </collision>
-            <inertial>
-                <mass value="0.2" />
-                <inertia ixx="0.4" ixy="0.0" ixz="0.0" iyy="0.4" iyz="0.0" izz="0.2" />
-            </inertial>
-            <origin xyz="0.01861 0 -0.02100" />
+        <inertial>
+            <mass value="1" />
+            <inertia ixx="0.1" ixy="0" ixz="0" iyy="0.1"
+                iyz="0" izz="0.1" />
+        </inertial>
+        <collision>
+            <geometry>
+                <mesh filename="file://$(find goddard_description)/meshes/tibia.stl"
+                    scale="0.001 0.001 0.001" />
+            </geometry>
+            <origin xyz="0.01861 0 -0.02100" rpy="0 0 0" />
+        </collision>
+        <visual>
+            <geometry>
+                <mesh filename="file://$(find goddard_description)/meshes/tibia.stl"
+                    scale="0.001 0.001 0.001" />
+            </geometry>
+            <origin xyz="0.01861 0 -0.02100" rpy="0 0 0" />
         </visual>
     </link>
@@ -165,5 +190,5 @@
         <parent link="front_right_femur" />
         <child link="front_right_tibia" />
-        <origin xyz="-0.05367 0 -0.05261" />
+        <origin xyz="-0.05367 0 -0.05261" rpy="0 0 0" />
         <axis xyz="0 -1 0" />
         <limit lower="-1.571" upper="1.571" effort="1000" velocity="0.5" />
@@ -171,17 +196,21 @@
     <!-- Back Left Components -->
     <link name="back_left_hip">
-        <visual>
-            <geometry>
-                <mesh filename="package://goddard_description/meshes/hip.stl"
-                    scale="0.001 0.001 0.001" />
-            </geometry>
-            <collision>
-                <mesh filename="package://goddard_description/meshes/hip.stl"
-                    scale="0.001 0.001 0.001" />
-            </collision>
-            <inertial>
-                <mass value="0.2" />
-                <inertia ixx="0.4" ixy="0.0" ixz="0.0" iyy="0.4" iyz="0.0" izz="0.2" />
-            </inertial>
+        <inertial>
+            <mass value="1" />
+            <inertia ixx="0.1" ixy="0" ixz="0" iyy="0.1"
+                iyz="0" izz="0.1" />
+        </inertial>
+        <collision>
+            <geometry>
+                <mesh filename="file://$(find goddard_description)/meshes/hip.stl"
+                    scale="0.001 0.001 0.001" />
+            </geometry>
+            <origin xyz="0 0 0" rpy="0 0 3.142" />
+        </collision>
+        <visual>
+            <geometry>
+                <mesh filename="file://$(find goddard_description)/meshes/hip.stl"
+                    scale="0.001 0.001 0.001" />
+            </geometry>
             <origin xyz="0 0 0" rpy="0 0 3.142" />
         </visual>
@@ -190,23 +219,27 @@
         <parent link="body" />
         <child link="back_left_hip" />
-        <origin xyz="-0.07900 0.05713 0.003000" />
+        <origin xyz="-0.07900 0.05713 0.003000" rpy="0 0 0" />
         <axis xyz="1 0 0" />
         <limit lower="-1.571" upper="1.571" effort="1000" velocity="0.5" />
     </joint>
     <link name="back_left_femur">
-        <visual>
-            <geometry>
-                <mesh filename="package://goddard_description/meshes/femur.stl"
-                    scale="0.001 0.001 0.001" />
-            </geometry>
-            <collision>
-                <mesh filename="package://goddard_description/meshes/femur.stl"
-                    scale="0.001 0.001 0.001" />
-            </collision>
-            <inertial>
-                <mass value="0.2" />
-                <inertia ixx="0.4" ixy="0.0" ixz="0.0" iyy="0.4" iyz="0.0" izz="0.2" />
-            </inertial>
-            <origin xyz="-0.0246 0 -0.02835" />
+        <inertial>
+            <mass value="1" />
+            <inertia ixx="0.1" ixy="0" ixz="0" iyy="0.1"
+                iyz="0" izz="0.1" />
+        </inertial>
+        <collision>
+            <geometry>
+                <mesh filename="file://$(find goddard_description)/meshes/femur.stl"
+                    scale="0.001 0.001 0.001" />
+            </geometry>
+            <origin xyz="-0.0246 0 -0.02835" rpy="0 0 0" />
+        </collision>
+        <visual>
+            <geometry>
+                <mesh filename="file://$(find goddard_description)/meshes/femur.stl"
+                    scale="0.001 0.001 0.001" />
+            </geometry>
+            <origin xyz="-0.0246 0 -0.02835" rpy="0 0 0" />
         </visual>
     </link>
@@ -214,23 +247,27 @@
         <parent link="back_left_hip" />
         <child link="back_left_femur" />
-        <origin xyz="0 0.03558 -0.00469" />
+        <origin xyz="0 0.03558 -0.00469" rpy="0 0 0" />
         <axis xyz="0 -1 0" />
         <limit lower="-1.571" upper="1.571" effort="1000" velocity="0.5" />
     </joint>
     <link name="back_left_tibia">
-        <visual>
-            <geometry>
-                <mesh filename="package://goddard_description/meshes/tibia.stl"
-                    scale="0.001 0.001 0.001" />
-            </geometry>
-            <collision>
-                <mesh filename="package://goddard_description/meshes/tibia.stl"
-                    scale="0.001 0.001 0.001" />
-            </collision>
-            <inertial>
-                <mass value="0.2" />
-                <inertia ixx="0.4" ixy="0.0" ixz="0.0" iyy="0.4" iyz="0.0" izz="0.2" />
-            </inertial>
-            <origin xyz="0.01861 0 -0.02100" />
+        <inertial>
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