Commit message: got major ros2 control components working. gazebo sim runs and broadcasts joint states. Want to work now on getting logic of a quadruped in sim, then make the hardware interface work

File: src/Goddard/goddard_description/urdf/goddard.urdf.xacro (robot description, xacro)
@@ -27,82 +27,82 @@
     </joint>
     <!-- Front Left Components  -->
-    <link name="front_left_hip">
-        <inertial>
-            <mass value="1" />
-            <inertia ixx="0.1" ixy="0" ixz="0" iyy="0.1"
-                iyz="0" izz="0.1" />
-        </inertial>
-        <collision>
-            <geometry>
-                <mesh filename="file://$(find goddard_description)/meshes/hip.stl"
-                    scale="0.001 0.001 0.001" />
-            </geometry>
-        </collision>
-        <visual>
-            <geometry>
-                <mesh filename="file://$(find goddard_description)/meshes/hip.stl"
-                    scale="0.001 0.001 0.001" />
-            </geometry>
-        </visual>
-    </link>
-    <joint name="front_left_hip_to_body" type="revolute">
+    <link name="fl_hip">
+        <inertial>
+            <mass value="1" />
+            <inertia ixx="0.1" ixy="0" ixz="0" iyy="0.1"
+                iyz="0" izz="0.1" />
+        </inertial>
+        <collision>
+            <geometry>
+                <mesh filename="file://$(find goddard_description)/meshes/hip.stl"
+                    scale="0.001 0.001 0.001" />
+            </geometry>
+        </collision>
+        <visual>
+            <geometry>
+                <mesh filename="file://$(find goddard_description)/meshes/hip.stl"
+                    scale="0.001 0.001 0.001" />
+            </geometry>
+        </visual>
+    </link>
+    <joint name="fl_hip_to_body" type="revolute">
         <parent link="body" />
-        <child link="front_left_hip" />
+        <child link="fl_hip" />
         <origin xyz="0.07900 0.05713 0.003000" rpy="0 0 0" />
         <axis xyz="1 0 0" />
         <limit lower="-1.571" upper="1.571" effort="1000" velocity="0.5" />
     </joint>
-    <link name="front_left_femur">
-        <inertial>
-            <mass value="1" />
-            <inertia ixx="0.1" ixy="0" ixz="0" iyy="0.1"
-                iyz="0" izz="0.1" />
-        </inertial>
-        <collision>
-            <geometry>
-                <mesh filename="file://$(find goddard_description)/meshes/femur.stl"
-                    scale="0.001 0.001 0.001" />
-            </geometry>
-            <origin xyz="-0.0246 0 -0.02835" rpy="0 0 0" />
-        </collision>
-        <visual>
-            <geometry>
-                <mesh filename="file://$(find goddard_description)/meshes/femur.stl"
-                    scale="0.001 0.001 0.001" />
-            </geometry>
-            <origin xyz="-0.0246 0 -0.02835" rpy="0 0 0" />
-        </visual>
-    </link>
-    <joint name="front_left_femur_to_front_left_hip" type="revolute">
-        <parent link="front_left_hip" />
-        <child link="front_left_femur" />
+    <link name="fl_femur">
+        <inertial>
+            <mass value="1" />
+            <inertia ixx="0.1" ixy="0" ixz="0" iyy="0.1"
+                iyz="0" izz="0.1" />
+        </inertial>
+        <collision>
+            <geometry>
+                <mesh filename="file://$(find goddard_description)/meshes/femur.stl"
+                    scale="0.001 0.001 0.001" />
+            </geometry>
+            <origin xyz="-0.0246 0 -0.02835" rpy="0 0 0" />
+        </collision>
+        <visual>
+            <geometry>
+                <mesh filename="file://$(find goddard_description)/meshes/femur.stl"
+                    scale="0.001 0.001 0.001" />
+            </geometry>
+            <origin xyz="-0.0246 0 -0.02835" rpy="0 0 0" />
+        </visual>
+    </link>
+    <joint name="fl_femur_to_hip" type="revolute">
+        <parent link="fl_hip" />
+        <child link="fl_femur" />
         <origin xyz="0 0.03558 -0.00469" rpy="0 0 0" />
         <axis xyz="0 -1 0" />
         <limit lower="-1.571" upper="1.571" effort="1000" velocity="0.5" />
     </joint>
-    <link name="front_left_tibia">
-        <inertial>
-            <mass value="1" />
-            <inertia ixx="0.1" ixy="0" ixz="0" iyy="0.1"
-                iyz="0" izz="0.1" />
-        </inertial>
-        <collision>
-            <geometry>
-                <mesh filename="file://$(find goddard_description)/meshes/tibia.stl"
-                    scale="0.001 0.001 0.001" />
-            </geometry>
-            <origin xyz="0.01861 0 -0.02100" rpy="0 0 0" />
-        </collision>
-        <visual>
-            <geometry>
-                <mesh filename="file://$(find goddard_description)/meshes/tibia.stl"
-                    scale="0.001 0.001 0.001" />
-            </geometry>
-            <origin xyz="0.01861 0 -0.02100" rpy="0 0 0" />
-        </visual>
-    </link>
-    <joint name="front_left_tibia_to_front_left_femur" type="revolute">
-        <parent link="front_left_femur" />
-        <child link="front_left_tibia" />
+    <link name="fl_tibia">
+        <inertial>
+            <mass value="1" />
+            <inertia ixx="0.1" ixy="0" ixz="0" iyy="0.1"
+                iyz="0" izz="0.1" />
+        </inertial>
+        <collision>
+            <geometry>
+                <mesh filename="file://$(find goddard_description)/meshes/tibia.stl"
+                    scale="0.001 0.001 0.001" />
+            </geometry>
+            <origin xyz="0.01861 0 -0.02100" rpy="0 0 0" />
+        </collision>
+        <visual>
+            <geometry>
+                <mesh filename="file://$(find goddard_description)/meshes/tibia.stl"
+                    scale="0.001 0.001 0.001" />
+            </geometry>
+            <origin xyz="0.01861 0 -0.02100" rpy="0 0 0" />
+        </visual>
+    </link>
+    <joint name="fl_tibia_to_femur" type="revolute">
+        <parent link="fl_femur" />
+        <child link="fl_tibia" />
         <origin xyz="-0.05367 0 -0.05261" rpy="0 0 0" />
         <axis xyz="0 -1 0" />
@@ -110,84 +110,84 @@
     </joint>
     <!-- Front Right Components -->
-    <link name="front_right_hip">
-        <inertial>
-            <mass value="1" />
-            <inertia ixx="0.1" ixy="0" ixz="0" iyy="0.1"
-                iyz="0" izz="0.1" />
-        </inertial>
-        <collision>
-            <geometry>
-                <mesh filename="file://$(find goddard_description)/meshes/hip.stl"
-                    scale="0.001 0.001 0.001" />
-            </geometry>
-            <origin xyz="0 0 0" rpy="0 0 3.142" />
-        </collision>
-        <visual>
-            <geometry>
-                <mesh filename="file://$(find goddard_description)/meshes/hip.stl"
-                    scale="0.001 0.001 0.001" />
-            </geometry>
-            <origin xyz="0 0 0" rpy="0 0 3.142" />
-        </visual>
-    </link>
-    <joint name="front_right_hip_to_body" type="revolute">
+    <link name="fr_hip">
+        <inertial>
+            <mass value="1" />
+            <inertia ixx="0.1" ixy="0" ixz="0" iyy="0.1"
+                iyz="0" izz="0.1" />
+        </inertial>
+        <collision>
+            <geometry>
+                <mesh filename="file://$(find goddard_description)/meshes/hip.stl"
+                    scale="0.001 0.001 0.001" />
+            </geometry>
+            <origin xyz="0 0 0" rpy="0 0 3.142" />
+        </collision>
+        <visual>
+            <geometry>
+                <mesh filename="file://$(find goddard_description)/meshes/hip.stl"
+                    scale="0.001 0.001 0.001" />
+            </geometry>
+            <origin xyz="0 0 0" rpy="0 0 3.142" />
+        </visual>
+    </link>
+    <joint name="fr_hip_to_body" type="revolute">
         <parent link="body" />
-        <child link="front_right_hip" />
+        <child link="fr_hip" />
         <origin xyz="0.07900 -0.05713 0.003000" rpy="0 0 0" />
         <axis xyz="-1 0 0" />
         <limit lower="-1.571" upper="1.571" effort="1000" velocity="0.5" />
     </joint>
-    <link name="front_right_femur">
-        <inertial>
-            <mass value="1" />
-            <inertia ixx="0.1" ixy="0" ixz="0" iyy="0.1"
-                iyz="0" izz="0.1" />
-        </inertial>
-        <collision>
-            <geometry>
-                <mesh filename="file://$(find goddard_description)/meshes/femur.stl"
-                    scale="0.001 0.001 0.001" />
-            </geometry>
-            <origin xyz="-0.0246 0 -0.02835" rpy="0 0 0" />
-        </collision>
-        <visual>
-            <geometry>
-                <mesh filename="file://$(find goddard_description)/meshes/femur.stl"
-                    scale="0.001 0.001 0.001" />
-            </geometry>
-            <origin xyz="-0.0246 0 -0.02835" rpy="0 0 0" />
-        </visual>
-    </link>
-    <joint name="front_right_femur_to_front_right_hip" type="revolute">
-        <parent link="front_right_hip" />
-        <child link="front_right_femur" />
+    <link name="fr_femur">
+        <inertial>
+            <mass value="1" />
+            <inertia ixx="0.1" ixy="0" ixz="0" iyy="0.1"
+                iyz="0" izz="0.1" />
+        </inertial>
+        <collision>
+            <geometry>
+                <mesh filename="file://$(find goddard_description)/meshes/femur.stl"
+                    scale="0.001 0.001 0.001" />
+            </geometry>
+            <origin xyz="-0.0246 0 -0.02835" rpy="0 0 0" />
+        </collision>
+        <visual>
+            <geometry>
+                <mesh filename="file://$(find goddard_description)/meshes/femur.stl"
+                    scale="0.001 0.001 0.001" />
+            </geometry>
+            <origin xyz="-0.0246 0 -0.02835" rpy="0 0 0" />
+        </visual>
+    </link>
+    <joint name="fr_femur_to_hip" type="revolute">
+        <parent link="fr_hip" />
+        <child link="fr_femur" />
         <origin xyz="0 -0.03558 -0.00469" rpy="0 0 0" />
         <axis xyz="0 -1 0" />
         <limit lower="-1.571" upper="1.571" effort="1000" velocity="0.5" />
     </joint>
-    <link name="front_right_tibia">
-        <inertial>
-            <mass value="1" />
-            <inertia ixx="0.1" ixy="0" ixz="0" iyy="0.1"
-                iyz="0" izz="0.1" />
-        </inertial>
-        <collision>
-            <geometry>
-                <mesh filename="file://$(find goddard_description)/meshes/tibia.stl"
-                    scale="0.001 0.001 0.001" />
-            </geometry>
-            <origin xyz="0.01861 0 -0.02100" rpy="0 0 0" />
-        </collision>
-        <visual>
-            <geometry>
-                <mesh filename="file://$(find goddard_description)/meshes/tibia.stl"
-                    scale="0.001 0.001 0.001" />
-            </geometry>
-            <origin xyz="0.01861 0 -0.02100" rpy="0 0 0" />
-        </visual>
-    </link>
-    <joint name="front_right_tibia_to_front_right_femur" type="revolute">
-        <parent link="front_right_femur" />
-        <child link="front_right_tibia" />
+    <link name="fr_tibia">
+        <inertial>
+            <mass value="1" />
+            <inertia ixx="0.1" ixy="0" ixz="0" iyy="0.1"
+                iyz="0" izz="0.1" />
+        </inertial>
+        <collision>
+            <geometry>
+                <mesh filename="file://$(find goddard_description)/meshes/tibia.stl"
+                    scale="0.001 0.001 0.001" />
+            </geometry>
+            <origin xyz="0.01861 0 -0.02100" rpy="0 0 0" />
+        </collision>
+        <visual>
+            <geometry>
+                <mesh filename="file://$(find goddard_description)/meshes/tibia.stl"
+                    scale="0.001 0.001 0.001" />
+            </geometry>
+            <origin xyz="0.01861 0 -0.02100" rpy="0 0 0" />
+        </visual>
+    </link>
+    <joint name="fr_tibia_to_femur" type="revolute">
+        <parent link="fr_femur" />
+        <child link="fr_tibia" />
         <origin xyz="-0.05367 0 -0.05261" rpy="0 0 0" />
         <axis xyz="0 -1 0" />
@@ -195,84 +195,84 @@
     </joint>
     <!-- Back Left Components -->
-    <link name="back_left_hip">
-        <inertial>
-            <mass value="1" />
-            <inertia ixx="0.1" ixy="0" ixz="0" iyy="0.1"
-                iyz="0" izz="0.1" />
-        </inertial>
-        <collision>
-            <geometry>
-                <mesh filename="file://$(find goddard_description)/meshes/hip.stl"
-                    scale="0.001 0.001 0.001" />
-            </geometry>
-            <origin xyz="0 0 0" rpy="0 0 3.142" />
-        </collision>
-        <visual>
-            <geometry>
-                <mesh filename="file://$(find goddard_description)/meshes/hip.stl"
-                    scale="0.001 0.001 0.001" />
-            </geometry>
-            <origin xyz="0 0 0" rpy="0 0 3.142" />
-        </visual>
-    </link>
-    <joint name="back_left_hip_to_body" type="revolute">
+    <link name="bl_hip">
+        <inertial>
+            <mass value="1" />
+            <inertia ixx="0.1" ixy="0" ixz="0" iyy="0.1"
+                iyz="0" izz="0.1" />
+        </inertial>
+        <collision>
+            <geometry>
+                <mesh filename="file://$(find goddard_description)/meshes/hip.stl"
+                    scale="0.001 0.001 0.001" />
+            </geometry>
+            <origin xyz="0 0 0" rpy="0 0 3.142" />
+        </collision>
+        <visual>
+            <geometry>
+                <mesh filename="file://$(find goddard_description)/meshes/hip.stl"
+                    scale="0.001 0.001 0.001" />
+            </geometry>
+            <origin xyz="0 0 0" rpy="0 0 3.142" />
+        </visual>
+    </link>
+    <joint name="bl_hip_to_body" type="revolute">
         <parent link="body" />
-        <child link="back_left_hip" />
+        <child link="bl_hip" />
         <origin xyz="-0.07900 0.05713 0.003000" rpy="0 0 0" />
         <axis xyz="1 0 0" />
         <limit lower="-1.571" upper="1.571" effort="1000" velocity="0.5" />
     </joint>
-    <link name="back_left_femur">
-        <inertial>
-            <mass value="1" />
-            <inertia ixx="0.1" ixy="0" ixz="0" iyy="0.1"
-                iyz="0" izz="0.1" />
-        </inertial>
-        <collision>
-            <geometry>
-                <mesh filename="file://$(find goddard_description)/meshes/femur.stl"
-                    scale="0.001 0.001 0.001" />
-            </geometry>
-            <origin xyz="-0.0246 0 -0.02835" rpy="0 0 0" />
-        </collision>
-        <visual>
-            <geometry>
-                <mesh filename="file://$(find goddard_description)/meshes/femur.stl"
-                    scale="0.001 0.001 0.001" />
-            </geometry>
-            <origin xyz="-0.0246 0 -0.02835" rpy="0 0 0" />
-        </visual>
-    </link>
-    <joint name="back_left_femur_to_back_left_hip" type="revolute">
-        <parent link="back_left_hip" />
-        <child link="back_left_femur" />
+    <link name="bl_femur">
+        <inertial>
+            <mass value="1" />
+            <inertia ixx="0.1" ixy="0" ixz="0" iyy="0.1"
+                iyz="0" izz="0.1" />
+        </inertial>
+        <collision>
+            <geometry>
+                <mesh filename="file://$(find goddard_description)/meshes/femur.stl"
+                    scale="0.001 0.001 0.001" />
+            </geometry>
+            <origin xyz="-0.0246 0 -0.02835" rpy="0 0 0" />
+        </collision>
+        <visual>
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