Commit message: starting to write the kinematics math myself, also realized that the urdf is wrong and that the femur and tibia are off by 45 deg due to the stls comming in that way, need to offset the visual and change joint locations

File: src/Goddard/goddard_description/urdf/goddard.urdf.xacro (robot description, xacro)
@@ -78,5 +78,5 @@
         <child link="fl_femur" />
         <origin xyz="0 0.03558 -0.00469" rpy="0 0 0" />
-        <axis xyz="0 -1 0" />
+        <axis xyz="0 1 0" />
         <limit lower="-1.571" upper="1.571" effort="1000" velocity="0.5" />
     </joint>
@@ -109,4 +109,10 @@
         <limit lower="-1.571" upper="1.571" effort="1000" velocity="0.5" />
     </joint>
+    <link name="fl_foot" />
+    <joint name="fl_foot_to_tibia" type="fixed">
+        <parent link="fl_tibia" />
+        <child link="fl_foot" />
+        <origin xyz="0.05367 0 -0.0543" rpy="0 0 0" />
+    </joint>
     <!-- Front Right Components -->
     <link name="fr_hip">
@@ -121,12 +127,12 @@
                     scale="0.001 0.001 0.001" />
             </geometry>
-            <origin xyz="0 0 0" rpy="0 0 3.142" />
-        </collision>
-        <visual>
-            <geometry>
-                <mesh filename="file://$(find goddard_description)/meshes/hip.stl"
-                    scale="0.001 0.001 0.001" />
-            </geometry>
-            <origin xyz="0 0 0" rpy="0 0 3.142" />
+            <origin xyz="0 0 0" rpy="0 0 0" />
+        </collision>
+        <visual>
+            <geometry>
+                <mesh filename="file://$(find goddard_description)/meshes/hip.stl"
+                    scale="0.001 0.001 0.001" />
+            </geometry>
+            <origin xyz="0 0 0" rpy="0 0 0" />
         </visual>
     </link>
@@ -134,6 +140,6 @@
         <parent link="body" />
         <child link="fr_hip" />
-        <origin xyz="0.07900 -0.05713 0.003000" rpy="0 0 0" />
-        <axis xyz="-1 0 0" />
+        <origin xyz="0.07900 -0.05713 0.003000" rpy="0 0 3.142" />
+        <axis xyz="1 0 0" />
         <limit lower="-1.571" upper="1.571" effort="1000" velocity="0.5" />
     </joint>
@@ -149,12 +155,12 @@
                     scale="0.001 0.001 0.001" />
             </geometry>
-            <origin xyz="-0.0246 0 -0.02835" rpy="0 0 0" />
-        </collision>
-        <visual>
-            <geometry>
-                <mesh filename="file://$(find goddard_description)/meshes/femur.stl"
-                    scale="0.001 0.001 0.001" />
-            </geometry>
-            <origin xyz="-0.0246 0 -0.02835" rpy="0 0 0" />
+            <origin xyz="0.0246 0 -0.02835" rpy="0 -1.571 0" />
+        </collision>
+        <visual>
+            <geometry>
+                <mesh filename="file://$(find goddard_description)/meshes/femur.stl"
+                    scale="0.001 0.001 0.001" />
+            </geometry>
+            <origin xyz="0.0246 0 -0.02835" rpy="0 -1.571 0" />
         </visual>
     </link>
@@ -162,6 +168,6 @@
         <parent link="fr_hip" />
         <child link="fr_femur" />
-        <origin xyz="0 -0.03558 -0.00469" rpy="0 0 0" />
-        <axis xyz="0 -1 0" />
+        <origin xyz="0 0.03558 -0.00469" rpy="0 0 0" />
+        <axis xyz="0 1 0" />
         <limit lower="-1.571" upper="1.571" effort="1000" velocity="0.5" />
     </joint>
@@ -177,12 +183,12 @@
                     scale="0.001 0.001 0.001" />
             </geometry>
-            <origin xyz="0.01861 0 -0.02100" rpy="0 0 0" />
-        </collision>
-        <visual>
-            <geometry>
-                <mesh filename="file://$(find goddard_description)/meshes/tibia.stl"
-                    scale="0.001 0.001 0.001" />
-            </geometry>
-            <origin xyz="0.01861 0 -0.02100" rpy="0 0 0" />
+            <origin xyz="-0.01861 0 -0.02100" rpy="0 0 3.142" />
+        </collision>
+        <visual>
+            <geometry>
+                <mesh filename="file://$(find goddard_description)/meshes/tibia.stl"
+                    scale="0.001 0.001 0.001" />
+            </geometry>
+            <origin xyz="-0.01861 0 -0.02100" rpy="0 0 3.142" />
         </visual>
     </link>
@@ -190,7 +196,13 @@
         <parent link="fr_femur" />
         <child link="fr_tibia" />
-        <origin xyz="-0.05367 0 -0.05261" rpy="0 0 0" />
-        <axis xyz="0 -1 0" />
-        <limit lower="-1.571" upper="1.571" effort="1000" velocity="0.5" />
+        <origin xyz="0.05367 0 -0.05261" rpy="0 0 0" />
+        <axis xyz="0 1 0" />
+        <limit lower="-1.571" upper="1.571" effort="1000" velocity="0.5" />
+    </joint>
+    <link name="fr_foot" />
+    <joint name="fr_foot_to_tibia" type="fixed">
+        <parent link="fr_tibia" />
+        <child link="fr_foot" />
+        <origin xyz="-0.05367 0 -0.0543" rpy="0 0 0" />
     </joint>
     <!-- Back Left Components -->
@@ -276,6 +288,12 @@
         <child link="bl_tibia" />
         <origin xyz="-0.05367 0 -0.05261" rpy="0 0 0" />
-        <axis xyz="0 -1 0" />
-        <limit lower="-1.571" upper="1.571" effort="1000" velocity="0.5" />
+        <axis xyz="0 1 0" />
+        <limit lower="-1.571" upper="1.571" effort="1000" velocity="0.5" />
+    </joint>
+    <link name="bl_foot" />
+    <joint name="bl_foot_to_tibia" type="fixed">
+        <parent link="bl_tibia" />
+        <child link="bl_foot" />
+        <origin xyz="0.05367 0 -0.0543" rpy="0 0 0" />
     </joint>
     <!-- Back Right Components -->
@@ -291,12 +309,12 @@
                     scale="0.001 0.001 0.001" />
             </geometry>
-            <origin xyz="0 0 0" rpy="0 0 3.142" />
-        </collision>
-        <visual>
-            <geometry>
-                <mesh filename="file://$(find goddard_description)/meshes/hip.stl"
-                    scale="0.001 0.001 0.001" />
-            </geometry>
-            <origin xyz="0 0 0" rpy="0 0 3.142" />
+            <origin xyz="0 0 0" rpy="0 0 0" />
+        </collision>
+        <visual>
+            <geometry>
+                <mesh filename="file://$(find goddard_description)/meshes/hip.stl"
+                    scale="0.001 0.001 0.001" />
+            </geometry>
+            <origin xyz="0 0 0" rpy="0 0 0" />
         </visual>
     </link>
@@ -304,6 +322,6 @@
         <parent link="body" />
         <child link="br_hip" />
-        <origin xyz="-0.07900 -0.05713 0.003000" rpy="0 0 0" />
-        <axis xyz="-1 0 0" />
+        <origin xyz="-0.07900 -0.05713 0.003000" rpy="0 0 3.142" />
+        <axis xyz="1 0 0" />
         <limit lower="-1.571" upper="1.571" effort="1000" velocity="0.5" />
     </joint>
@@ -319,12 +337,12 @@
                     scale="0.001 0.001 0.001" />
             </geometry>
-            <origin xyz="-0.0246 0 -0.02835" rpy="0 0 0" />
-        </collision>
-        <visual>
-            <geometry>
-                <mesh filename="file://$(find goddard_description)/meshes/femur.stl"
-                    scale="0.001 0.001 0.001" />
-            </geometry>
-            <origin xyz="-0.0246 0 -0.02835" rpy="0 0 0" />
+            <origin xyz="0.0246 0 -0.02835" rpy="0 -1.571 0" />
+        </collision>
+        <visual>
+            <geometry>
+                <mesh filename="file://$(find goddard_description)/meshes/femur.stl"
+                    scale="0.001 0.001 0.001" />
+            </geometry>
+            <origin xyz="0.0246 0 -0.02835" rpy="0 -1.571 0" />
         </visual>
     </link>
@@ -332,6 +350,6 @@
         <parent link="br_hip" />
         <child link="br_femur" />
-        <origin xyz="0 -0.03558 -0.00469" rpy="0 0 0" />
-        <axis xyz="0 -1 0" />
+        <origin xyz="0 0.03558 -0.00469" rpy="0 0 0" />
+        <axis xyz="0 1 0" />
         <limit lower="-1.571" upper="1.571" effort="1000" velocity="0.5" />
     </joint>
@@ -347,12 +365,12 @@
                     scale="0.001 0.001 0.001" />
             </geometry>
-            <origin xyz="0.01861 0 -0.02100" rpy="0 0 0" />
-        </collision>
-        <visual>
-            <geometry>
-                <mesh filename="file://$(find goddard_description)/meshes/tibia.stl"
-                    scale="0.001 0.001 0.001" />
-            </geometry>
-            <origin xyz="0.01861 0 -0.02100" rpy="0 0 0" />
+            <origin xyz="-0.01861 0 -0.02100" rpy="0 0 3.142" />
+        </collision>
+        <visual>
+            <geometry>
+                <mesh filename="file://$(find goddard_description)/meshes/tibia.stl"
+                    scale="0.001 0.001 0.001" />
+            </geometry>
+            <origin xyz="-0.01861 0 -0.02100" rpy="0 0 3.142" />
         </visual>
     </link>
@@ -360,7 +378,13 @@
         <parent link="br_femur" />
         <child link="br_tibia" />
-        <origin xyz="-0.05367 0 -0.05261" rpy="0 0 0" />
-        <axis xyz="0 -1 0" />
-        <limit lower="-1.571" upper="1.571" effort="1000" velocity="0.5" />
+        <origin xyz="0.05367 0 -0.05261" rpy="0 0 0" />
+        <axis xyz="0 1 0" />
+        <limit lower="-1.571" upper="1.571" effort="1000" velocity="0.5" />
+    </joint>
+    <link name="br_foot" />
+    <joint name="br_foot_to_tibia" type="fixed">
+        <parent link="br_tibia" />
+        <child link="br_foot" />
+        <origin xyz="-0.05367 0 -0.0543" rpy="0 0 0" />
     </joint>
     <xacro:include filename="ros2_control.xacro" />
