Commit message: fixed front right leg, need to do the rest

File: src/Goddard/goddard_description/urdf/robot_core.xacro (robot description, xacro)
@@ -38,10 +38,12 @@
                     scale="0.001 0.001 0.001" />
             </geometry>
-        </collision>
-        <visual>
-            <geometry>
-                <mesh filename="file://$(find goddard_description)/meshes/hip.stl"
-                    scale="0.001 0.001 0.001" />
-            </geometry>
+            <origin xyz="0 0 0" rpy="0 0 0" />
+        </collision>
+        <visual>
+            <geometry>
+                <mesh filename="file://$(find goddard_description)/meshes/hip.stl"
+                    scale="0.001 0.001 0.001" />
+            </geometry>
+            <origin xyz="0 0 0" rpy="0 0 0" />
         </visual>
     </link>
@@ -155,12 +157,12 @@
                     scale="0.001 0.001 0.001" />
             </geometry>
-            <origin xyz="0.0246 0 -0.02835" rpy="0 -1.571 0" />
-        </collision>
-        <visual>
-            <geometry>
-                <mesh filename="file://$(find goddard_description)/meshes/femur.stl"
-                    scale="0.001 0.001 0.001" />
-            </geometry>
-            <origin xyz="0.0246 0 -0.02835" rpy="0 -1.571 0" />
+            <origin xyz="0 0 -0.03806" rpy="0 0.785398 0" />
+        </collision>
+        <visual>
+            <geometry>
+                <mesh filename="file://$(find goddard_description)/meshes/femur.stl"
+                    scale="0.001 0.001 0.001" />
+            </geometry>
+            <origin xyz="0 0 -0.03806" rpy="0 -0.785398 0" />
         </visual>
     </link>
@@ -168,5 +170,5 @@
         <parent link="fr_hip" />
         <child link="fr_femur" />
-        <origin xyz="0 0.03558 -0.00469" rpy="0 0 0" />
+        <origin xyz="0 0.03558 -0.00300" rpy="0 0 0" />
         <axis xyz="0 1 0" />
         <limit lower="-1.571" upper="1.571" effort="1000" velocity="0.5" />
@@ -183,12 +185,12 @@
                     scale="0.001 0.001 0.001" />
             </geometry>
-            <origin xyz="-0.01861 0 -0.02100" rpy="0 0 3.142" />
-        </collision>
-        <visual>
-            <geometry>
-                <mesh filename="file://$(find goddard_description)/meshes/tibia.stl"
-                    scale="0.001 0.001 0.001" />
-            </geometry>
-            <origin xyz="-0.01861 0 -0.02100" rpy="0 0 3.142" />
+            <origin xyz="-0.0030 0 -0.03058" rpy="0 0.733038 3.142" />
+        </collision>
+        <visual>
+            <geometry>
+                <mesh filename="file://$(find goddard_description)/meshes/tibia.stl"
+                    scale="0.001 0.001 0.001" />
+            </geometry>
+            <origin xyz="-0.0030 0 -0.03058" rpy="0 0.733038 3.142" />
         </visual>
     </link>
@@ -196,5 +198,5 @@
         <parent link="fr_femur" />
         <child link="fr_tibia" />
-        <origin xyz="0.05367 0 -0.05261" rpy="0 0 0" />
+        <origin xyz="0 0 -0.07560" rpy="0 0 0" />
         <axis xyz="0 1 0" />
         <limit lower="-1.571" upper="1.571" effort="1000" velocity="0.5" />

Commit message: got the left side kinematics in a good spot, now i need to look into fixing the foot frame and working on rightside hip kinematics

File: src/Goddard/goddard_description/urdf/robot_core.xacro (robot description, xacro)
@@ -80,5 +80,5 @@
         <child link="fl_femur" />
         <origin xyz="0 0.03558 -0.00300" rpy="0 0 0" />
-        <axis xyz="0 1 0" />
+        <axis xyz="0 -1 0" />
         <limit lower="-1.571" upper="1.571" effort="1000" velocity="0.5" />
     </joint>
@@ -220,12 +220,12 @@
                     scale="0.001 0.001 0.001" />
             </geometry>
-            <origin xyz="0 0 0" rpy="0 0 3.142" />
-        </collision>
-        <visual>
-            <geometry>
-                <mesh filename="file://$(find goddard_description)/meshes/hip.stl"
-                    scale="0.001 0.001 0.001" />
-            </geometry>
-            <origin xyz="0 0 0" rpy="0 0 3.142" />
+            <origin xyz="0 0 0" rpy="0 0 0" />
+        </collision>
+        <visual>
+            <geometry>
+                <mesh filename="file://$(find goddard_description)/meshes/hip.stl"
+                    scale="0.001 0.001 0.001" />
+            </geometry>
+            <origin xyz="0 0 0" rpy="0 0 0" />
         </visual>
     </link>
@@ -248,12 +248,12 @@
                     scale="0.001 0.001 0.001" />
             </geometry>
-            <origin xyz="-0.0246 0 -0.02835" rpy="0 0 0" />
-        </collision>
-        <visual>
-            <geometry>
-                <mesh filename="file://$(find goddard_description)/meshes/femur.stl"
-                    scale="0.001 0.001 0.001" />
-            </geometry>
-            <origin xyz="-0.0246 0 -0.02835" rpy="0 0 0" />
+            <origin xyz="0 0 -0.03806" rpy="0 -0.785398 0" />
+        </collision>
+        <visual>
+            <geometry>
+                <mesh filename="file://$(find goddard_description)/meshes/femur.stl"
+                    scale="0.001 0.001 0.001" />
+            </geometry>
+            <origin xyz="-0 0 -0.03806" rpy="0 -0.785398 0" />
         </visual>
     </link>
@@ -261,5 +261,5 @@
         <parent link="bl_hip" />
         <child link="bl_femur" />
-        <origin xyz="0 0.03558 -0.00469" rpy="0 0 0" />
+        <origin xyz="0 0.03558 -0.00300" rpy="0 0 0" />
         <axis xyz="0 -1 0" />
         <limit lower="-1.571" upper="1.571" effort="1000" velocity="0.5" />
@@ -276,12 +276,12 @@
                     scale="0.001 0.001 0.001" />
             </geometry>
-            <origin xyz="0.01861 0 -0.02100" rpy="0 0 0" />
-        </collision>
-        <visual>
-            <geometry>
-                <mesh filename="file://$(find goddard_description)/meshes/tibia.stl"
-                    scale="0.001 0.001 0.001" />
-            </geometry>
-            <origin xyz="0.01861 0 -0.02100" rpy="0 0 0" />
+            <origin xyz="-0.0030 0 -0.03058" rpy="0 0.733038 0" />
+        </collision>
+        <visual>
+            <geometry>
+                <mesh filename="file://$(find goddard_description)/meshes/tibia.stl"
+                    scale="0.001 0.001 0.001" />
+            </geometry>
+            <origin xyz="-0.0030 0 -0.03058" rpy="0 0.733038 0" />
         </visual>
     </link>
@@ -289,6 +289,6 @@
         <parent link="bl_femur" />
         <child link="bl_tibia" />
-        <origin xyz="-0.05367 0 -0.05261" rpy="0 0 0" />
-        <axis xyz="0 1 0" />
+        <origin xyz="0 0 -0.07560" rpy="0 0 0" />
+        <axis xyz="0 -1 0" />
         <limit lower="-1.571" upper="1.571" effort="1000" velocity="0.5" />
     </joint>
@@ -339,12 +339,12 @@
                     scale="0.001 0.001 0.001" />
             </geometry>
-            <origin xyz="0.0246 0 -0.02835" rpy="0 -1.571 0" />
-        </collision>
-        <visual>
-            <geometry>
-                <mesh filename="file://$(find goddard_description)/meshes/femur.stl"
-                    scale="0.001 0.001 0.001" />
-            </geometry>
-            <origin xyz="0.0246 0 -0.02835" rpy="0 -1.571 0" />
+            <origin xyz="0 0 -0.03806" rpy="0 -0.785398 0" />
+        </collision>
+        <visual>
+            <geometry>
+                <mesh filename="file://$(find goddard_description)/meshes/femur.stl"
+                    scale="0.001 0.001 0.001" />
+            </geometry>
+            <origin xyz="0 0 -0.03806" rpy="0 -0.785398 0" />
         </visual>
     </link>
@@ -352,5 +352,5 @@
         <parent link="br_hip" />
         <child link="br_femur" />
-        <origin xyz="0 0.03558 -0.00469" rpy="0 0 0" />
+        <origin xyz="0 0.03558 -0.00300" rpy="0 0 0" />
         <axis xyz="0 1 0" />
         <limit lower="-1.571" upper="1.571" effort="1000" velocity="0.5" />
@@ -367,12 +367,12 @@
                     scale="0.001 0.001 0.001" />
             </geometry>
-            <origin xyz="-0.01861 0 -0.02100" rpy="0 0 3.142" />
-        </collision>
-        <visual>
-            <geometry>
-                <mesh filename="file://$(find goddard_description)/meshes/tibia.stl"
-                    scale="0.001 0.001 0.001" />
-            </geometry>
-            <origin xyz="-0.01861 0 -0.02100" rpy="0 0 3.142" />
+            <origin xyz="-0.0030 0 -0.03058" rpy="0 0.733038 3.142" />
+        </collision>
+        <visual>
+            <geometry>
+                <mesh filename="file://$(find goddard_description)/meshes/tibia.stl"
+                    scale="0.001 0.001 0.001" />
+            </geometry>
+            <origin xyz="-0.0030 0 -0.03058" rpy="0 0.733038 3.142" />
         </visual>
     </link>
@@ -380,5 +380,5 @@
         <parent link="br_femur" />
         <child link="br_tibia" />
-        <origin xyz="0.05367 0 -0.05261" rpy="0 0 0" />
+        <origin xyz="0 0 -0.07560" rpy="0 0 0" />
         <axis xyz="0 1 0" />
         <limit lower="-1.571" upper="1.571" effort="1000" velocity="0.5" />
